File: hardware/ATmega328-TQFP32/4chord-midi.kicad_pcb (KiCad board)
At the start: 2 copper layers, 85.6 x 54 mm, 60 parts, among them IC1 ATMEGA328P-A, P1 USB_B, P2 Programmer, P3 CONN_01X04, P4 Nokia 3310 LCD, P5 LCD Backlight, SW1 SW_PUSH, SW2 SW_PUSH, SW3 SW_PUSH, SW4 SW_PUSH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

Commit message: Added CERN OHL v.1.2 licensing documentation
Other:
- board text added: "Licensed under CERN OHL v.1.2"
Changed lines of the file:
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@@
-(kicad_pcb (version 4) (host pcbnew 4.0.1-2.201512121406+6195~38~ubuntu14.04.1-stable)
+(kicad_pcb (version 4) (host pcbnew 4.0.1-3.201512161002+6197~38~ubuntu14.04.1-stable)
   (general
     (links 125)
@@
     (area 103.524999 32.385 189.42262 89.055001)
     (thickness 1.6)
-    (drawings 41)
+    (drawings 42)
     (tracks 558)
     (zones 0)
@@
     (visible_elements FFFFFF7F)
     (pcbplotparams
-      (layerselection 0x030f0_80000001)
+      (layerselection 0x010f0_80000001)
       (usegerberextensions false)
       (excludeedgelayer true)
@@
       (xy -0.614942 2.889672) (xy -0.522655 3.382412) (xy 0.548183 3.382412) (xy 0.64047 2.889672)) (layer B.Mask) (width 0.002))
   )
+  (gr_text "Licensed under CERN OHL v.1.2" (at 136.6 87.2) (layer B.SilkS)
+    (effects (font (size 0.5 0.5) (thickness 0.1)) (justify mirror))
+  )
   (gr_line (start 186 35) (end 106.81 35) (layer Edge.Cuts) (width 0.15))
