File: hardware/ATmega328-TQFP32/4chord-midi.sch (KiCad schematic (older format))
At the start: 46 parts, among them IC1 ATMEGA328P-A, P1 USB_B, P2 Programmer, P3 CONN_01X04, P4 Nokia 3310 LCD, P5 LCD Backlight, SW1 SW_PUSH, SW2 SW_PUSH, SW3 SW_PUSH, SW4 SW_PUSH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

Commit message: issue-#1: fixed broken connection R4-GND
Connections:
- wire segments 185 -> 150
Changed lines of the file:
@@
 LIBS:contrib
 LIBS:valves
+LIBS:4chord-midi-cache
 EELAYER 25 0
 EELAYER END
@@
 	5950 1400 5550 1400
 Wire Wire Line
-	5550 950  5550 1400
-Wire Wire Line
-	5550 1400 5550 2150
-Wire Wire Line
-	5550 2450 5550 3200
-Wire Wire Line
-	5550 3200 5550 3550
+	5550 950  5550 2150
+Wire Wire Line
+	5550 2450 5550 3550
 Wire Wire Line
 	5550 3200 5950 3200
 Wire Wire Line
-	5300 950  5300 1200
-Wire Wire Line
-	5300 1200 5300 2150
+	5300 950  5300 2150
 Wire Wire Line
 	5300 1200 5950 1200
@@
 	5950 1100 5050 1100
 Wire Wire Line
-	5050 950  5050 1100
-Wire Wire Line
-	5050 1100 5050 2150
-Wire Wire Line
-	5050 2450 5050 3400
-Wire Wire Line
-	5050 3400 5050 3550
+	5050 950  5050 2150
+Wire Wire Line
+	5050 2450 5050 3550
 Wire Wire Line
 	5050 3400 5950 3400
@@
 	5950 3300 5300 3300
 Wire Wire Line
-	5300 2450 5300 3300
-Wire Wire Line
-	5300 3300 5300 3550
-Wire Wire Line
-	1350 1050 2800 1050
-Wire Wire Line
-	2800 1050 2950 1050
-Wire Wire Line
-	3750 1050 3900 1050
-Wire Wire Line
-	3900 1050 4150 1050
+	5300 2450 5300 3550
+Wire Wire Line
+	1350 1050 2950 1050
+Wire Wire Line
+	3750 1050 4150 1050
 Wire Wire Line
 	1350 1350 1500 1350
@@
 	950  1650 950  1550
 Wire Wire Line
-	3350 1350 3350 1600
-Wire Wire Line
-	3350 1600 3350 1700
-Wire Wire Line
-	3350 1700 3350 1800
+	3350 1350 3350 1800
 Wire Wire Line
 	4150 1050 4150 950
@@
 	2350 4250 2350 4300
 Wire Wire Line
-	1550 3850 1700 3850
-Wire Wire Line
-	1700 3850 1900 3850
+	1550 3850 1900 3850
 Wire Wire Line
 	1700 3850 1700 3950
 Wire Wire Line
-	2200 3850 2350 3850
-Wire Wire Line
-	2350 3850 2500 3850
+	2200 3850 2500 3850
 Wire Wire Line
 	2350 3850 2350 3950
@@
 	4150 4550 4300 4550
 Wire Wire Line
-	4900 4550 5100 4550
-Wire Wire Line
-	5100 4550 5350 4550
+	4900 4550 5350 4550
 Wire Wire Line
 	5100 4550 5100 4650
@@
 	4150 5350 4300 5350
 Wire Wire Line
-	4900 5350 5100 5350
-Wire Wire Line
-	5100 5350 5350 5350
+	4900 5350 5350 5350
 Wire Wire Line
 	5100 5350 5100 5450
@@
 	4150 6150 4300 6150
 Wire Wire Line
-	4900 6150 5100 6150
-Wire Wire Line
-	5100 6150 5350 6150
+	4900 6150 5350 6150
 Wire Wire Line
 	5100 6150 5100 6250
@@
 	4150 6950 4300 6950
 Wire Wire Line
-	4900 6950 5100 6950
-Wire Wire Line
-	5100 6950 5350 6950
+	4900 6950 5350 6950
 Wire Wire Line
 	5100 6950 5100 7050
@@
 	1200 5350 1350 5350
 Wire Wire Line
-	1950 5350 2150 5350
-Wire Wire Line
-	2150 5350 2400 5350
+	1950 5350 2400 5350
 Wire Wire Line
 	2150 5350 2150 5450
@@
 	1200 6150 1350 6150
 Wire Wire Line
-	1950 6150 2150 6150
-Wire Wire Line
-	2150 6150 2400 6150
+	1950 6150 2400 6150
 Wire Wire Line
 	2150 6150 2150 6250
@@
 	1200 6950 1350 6950
 Wire Wire Line
-	1950 6950 2150 6950
-Wire Wire Line
-	2150 6950 2400 6950
+	1950 6950 2400 6950
 Wire Wire Line
 	2150 6950 2150 7050
@@
 	10650 1700 10500 1700
 Wire Wire Line
-	10650 1400 10650 1500
-Wire Wire Line
-	10650 1500 10650 1600
-Wire Wire Line
-	10650 1600 10650 1700
-Wire Wire Line
-	10650 1700 10650 1750
+	10650 1400 10650 1750
 Wire Wire Line
 	10500 1600 10650 1600
@@
 LCD_D#C
 Wire Wire Line
-	7800 5050 9050 5050
-Wire Wire Line
-	9050 5050 9750 5050
+	7800 5050 9750 5050
 Text Label 7800 5150 2    60   ~ 0
 LCD_#CS
 Wire Wire Line
-	7800 5150 9250 5150
-Wire Wire Line
-	9250 5150 9750 5150
+	7800 5150 9750 5150
 $Comp
 L C C16
@@
 LCD_#RESET
 Wire Wire Line
-	7800 5450 9450 5450
-Wire Wire Line
-	9450 5450 9750 5450
+	7800 5450 9750 5450
 $Comp
 L C C15
@@
 Connection ~ 9050 5050
 Wire Wire Line
-	7950 4300 8700 4300
-Wire Wire Line
-	8700 4300 9050 4300
-Wire Wire Line
-	9050 4300 9250 4300
-Wire Wire Line
-	9250 4300 9450 4300
-Wire Wire Line
-	9450 4300 9650 4300
-Wire Wire Line
-	9650 4300 9900 4300
+	7950 4300 9900 4300
 Wire Wire Line
 	9650 4300 9650 4750
@@
 	9650 5900 9650 5250
 Wire Wire Line
-	7950 5900 8700 5900
-Wire Wire Line
-	8700 5900 9050 5900
-Wire Wire Line
-	9050 5900 9650 5900
-Wire Wire Line
-	9650 5900 10350 5900
+	7950 5900 10350 5900
 Wire Wire Line
 	8700 4750 8700 5900
@@
 L GND #PWR032
 U 1 1 5660F85F
-P 2050 3050
-F 0 "#PWR032" H 2050 2800 50  0001 C CNN
-F 1 "GND" H 2050 2900 50  0000 C CNN
-F 2 "" H 2050 3050 50  0000 C CNN
-F 3 "" H 2050 3050 50  0000 C CNN
-	1    2050 3050
-	1    0    0    -1
-$EndComp
-Wire Wire Line
-	2050 3050 2050 2950
+P 2050 3000
+F 0 "#PWR032" H 2050 2750 50  0001 C CNN
+F 1 "GND" H 2050 2850 50  0000 C CNN
+F 2 "" H 2050 3000 50  0000 C CNN
+F 3 "" H 2050 3000 50  0000 C CNN
+	1    2050 3000
+	1    0    0    -1
+$EndComp
 Text Label 2750 2550 0    60   ~ 0
 USB_RESET
@@
 	1350 1150 2200 1150
 Wire Wire Line
-	2200 1150 2200 2250
-Wire Wire Line
-	2200 2250 2200 2550
+	2200 1150 2200 2550
 Wire Wire Line
 	2200 2250 2300 2250
@@
 	1350 1250 2050 1250
 Wire Wire Line
-	2050 1250 2050 2400
-Wire Wire Line
-	2050 2400 2050 2600
+	2050 1250 2050 2600
 Wire Wire Line
 	2050 2400 2300 2400
@@
 Wire Wire Line
 	10000 3000 10200 3000
+Wire Wire Line
+	2050 3000 2050 2900
 $EndSCHEMATC

Commit message: issue-#1: Added test points and zero-Ohm links
Parts:
- added R16, R17, R18: 0R, symbol R
- added W1, W2, W3, W4, W5: TP, symbol TEST_1P
Connections:
- wire segments 150 -> 160
Other:
- moved on the sheet: C1, C2, C3, C4, C5, IC1, P1, R1, R2, R3, R4, U1

Commit message: issue-#1: Added ground test points / pins
Parts:
- added W10, W6, W7, W8, W9: TP, symbol TEST_1P
Connections:
- wire segments 160 -> 164

Commit message: issue-#2: Added component footprints
Parts:
- C1, C16, C2: footprint (none) -> Capacitors_Tantalum_SMD:TantalC_SizeA_EIA-3216_HandSoldering
- C10, C11, C12, C13, C14, C15, C3, C4, C5, C6, C7, C8, C9: footprint (none) -> Capacitors_SMD:C_0805_HandSoldering
- IC1: footprint TQFP32 -> Housings_QFP:TQFP-32_7x7mm_Pitch0.8mm
- P1: footprint (none) -> Connect:USB_Mini-B
- P2: footprint (none) -> Pin_Headers:Pin_Header_Straight_2x05
- P3: footprint (none) -> Pin_Headers:Pin_Header_Straight_1x04
- P4: footprint (none) -> LCD_Connectors:FPA-WZA201-08-LF
- P5: footprint (none) -> SMD_Packages:SMD-2512_Pol
- R1, R10, R11, R12, R13, R14, R15, R16, R17, R18, R2, R3, R4, R5, R6, R7, R8, R9: footprint (none) -> Resistors_SMD:R_0805_HandSoldering
- SW1, SW2, SW3, SW4, SW5, SW6, SW7: footprint (none) -> Buttons_Switches_SMD:SW_SPST_EVPBF
- U1: footprint SOT-223 -> TO_SOT_Packages_SMD:SOT-223
- W1, W2, W3, W4, W5: footprint (none) -> SMD_Packages:1Pin
- W10, W6, W7, W8, W9: footprint (none) -> Connect:1pin
- X1: footprint (none) -> Crystals:crystal_FA238-TSX3225

Commit message: issue-#2: Removed some grounding pins and changed footprints of remaining ones
Parts:
- removed W7, W8, W9: TP, Connect:1pin, symbol TEST_1P
- W6: footprint Connect:1pin -> Pin_Headers:Pin_Header_Straight_1x01
- W7: renamed from W10; footprint Connect:1pin -> Pin_Headers:Pin_Header_Straight_1x01
Connections:
- wire segments 164 -> 161
Changed lines of the file:
@@
 F 0 "W6" H 1400 2170 50  0000 C CNN
 F 1 "TP" H 1400 2100 50  0000 C CNN
-F 2 "Connect:1pin" H 1600 1900 50  0001 C CNN
+F 2 "Pin_Headers:Pin_Header_Straight_1x01" H 1600 1900 50  0001 C CNN
 F 3 "" H 1600 1900 50  0000 C CNN
 	1    1400 1900
 	0    -1   -1   0
-$EndComp
-$Comp
-L TEST_1P W9
-U 1 1 5661E423
-P 8250 5950
-F 0 "W9" H 8250 6220 50  0000 C CNN
-F 1 "TP" H 8250 6150 50  0000 C CNN
-F 2 "Connect:1pin" H 8450 5950 50  0001 C CNN
-F 3 "" H 8450 5950 50  0000 C CNN
-	1    8250 5950
-	-1   0    0    1
-$EndComp
-$Comp
-L TEST_1P W8
-U 1 1 5661E8C8
-P 5900 3500
-F 0 "W8" H 5900 3770 50  0000 C CNN
-F 1 "TP" H 5900 3700 50  0000 C CNN
-F 2 "Connect:1pin" H 6100 3500 50  0001 C CNN
-F 3 "" H 6100 3500 50  0000 C CNN
-	1    5900 3500
-	-1   0    0    1
 $EndComp
 Wire Wire Line
@@
 Wire Wire Line
 	3850 1450 3850 1700
-Wire Wire Line
-	3850 1700 3300 1700
 Connection ~ 3300 1700
 Wire Wire Line
@@
 	1400 1900 1450 1900
 Connection ~ 1450 1900
-Wire Wire Line
-	8250 5950 8250 5900
-Connection ~ 8250 5900
-Wire Wire Line
-	5900 3500 5900 3400
-Connection ~ 5900 3400
 $Comp
-L TEST_1P W10
+L TEST_1P W7
 U 1 1 5661EF26
 P 10750 1400
-F 0 "W10" H 10750 1670 50  0000 C CNN
+F 0 "W7" H 10750 1670 50  0000 C CNN
 F 1 "TP" H 10750 1600 50  0000 C CNN
-F 2 "Connect:1pin" H 10950 1400 50  0001 C CNN
+F 2 "Pin_Headers:Pin_Header_Straight_1x01" H 10950 1400 50  0001 C CNN
 F 3 "" H 10950 1400 50  0000 C CNN
 	1    10750 1400
@@
 $EndComp
 Connection ~ 10650 1400
-$Comp
-L TEST_1P W7
-U 1 1 5661F52E
-P 3500 1750
-F 0 "W7" H 3500 2020 50  0000 C CNN
-F 1 "TP" H 3500 1950 50  0000 C CNN
-F 2 "Connect:1pin" H 3700 1750 50  0001 C CNN
-F 3 "" H 3700 1750 50  0000 C CNN
-	1    3500 1750
-	-1   0    0    1
-$EndComp
-Wire Wire Line
-	3500 1750 3500 1700
-Connection ~ 3500 1700
+Wire Wire Line
+	3850 1700 3300 1700
 $EndSCHEMATC

Commit message: Added CERN OHL v.1.2 licensing documentation
Other:
- note added: "Copyright Sven Gregori 2015.\n\nThis documentation describes Open Hardware and is licensed under the\nCERN OHL v. 1.2. You may redistribute and modify this documentation\nunder the terms of the CERN OHL v.1.2. (http://ohwr.org/cernohl).\n\nThis documentation is distributed WITHOUT ANY EXPRESS OR IMPLIED\nWARRANTY, INCLUDING OF MERCHANTABILITY, SATISFACTORY QUALITY AND\nFITNESS FOR A PARTICULAR PU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"
- moved on the sheet: C6, C7, X1
Changed lines of the file:
@@
 L Crystal X1
 U 1 1 565F9FF1
-P 2050 3850
-F 0 "X1" H 2050 4000 50  0000 C CNN
-F 1 "16MHz" H 2050 3700 50  0000 C CNN
-F 2 "Crystals:crystal_FA238-TSX3225" H 2050 3850 50  0001 C CNN
-F 3 "" H 2050 3850 50  0000 C CNN
-	1    2050 3850
+P 1700 3950
+F 0 "X1" H 1700 4100 50  0000 C CNN
+F 1 "16MHz" H 1700 3800 50  0000 C CNN
+F 2 "Crystals:crystal_FA238-TSX3225" H 1700 3950 50  0001 C CNN
+F 3 "" H 1700 3950 50  0000 C CNN
+	1    1700 3950
 	1    0    0    -1
 $EndComp
@@
 L C C6
 U 1 1 565FA22F
-P 1700 4100
-F 0 "C6" H 1725 4200 50  0000 L CNN
-F 1 "27p" H 1725 4000 50  0000 L CNN
-F 2 "Capacitors_SMD:C_0805_HandSoldering" H 1738 3950 50  0001 C CNN
-F 3 "" H 1700 4100 50  0000 C CNN
-	1    1700 4100
+P 1350 4200
+F 0 "C6" H 1375 4300 50  0000 L CNN
+F 1 "27p" H 1375 4100 50  0000 L CNN
+F 2 "Capacitors_SMD:C_0805_HandSoldering" H 1388 4050 50  0001 C CNN
+F 3 "" H 1350 4200 50  0000 C CNN
+	1    1350 4200
 	1    0    0    -1
 $EndComp
@@
 L C C7
 U 1 1 565FA29A
-P 2350 4100
-F 0 "C7" H 2375 4200 50  0000 L CNN
-F 1 "27p" H 2375 4000 50  0000 L CNN
-F 2 "Capacitors_SMD:C_0805_HandSoldering" H 2388 3950 50  0001 C CNN
-F 3 "" H 2350 4100 50  0000 C CNN
-	1    2350 4100
+P 2000 4200
+F 0 "C7" H 2025 4300 50  0000 L CNN
+F 1 "27p" H 2025 4100 50  0000 L CNN
+F 2 "Capacitors_SMD:C_0805_HandSoldering" H 2038 4050 50  0001 C CNN
+F 3 "" H 2000 4200 50  0000 C CNN
+	1    2000 4200
 	1    0    0    -1
 $EndComp
@@
 L GND #PWR012
 U 1 1 565FA355
-P 1700 4300
-F 0 "#PWR012" H 1700 4050 50  0001 C CNN
-F 1 "GND" H 1700 4150 50  0000 C CNN
-F 2 "" H 1700 4300 50  0000 C CNN
-F 3 "" H 1700 4300 50  0000 C CNN
-	1    1700 4300
+P 1350 4400
+F 0 "#PWR012" H 1350 4150 50  0001 C CNN
+F 1 "GND" H 1350 4250 50  0000 C CNN
+F 2 "" H 1350 4400 50  0000 C CNN
+F 3 "" H 1350 4400 50  0000 C CNN
+	1    1350 4400
 	1    0    0    -1
 $EndComp
@@
 L GND #PWR013
 U 1 1 565FA396
-P 2350 4300
-F 0 "#PWR013" H 2350 4050 50  0001 C CNN
-F 1 "GND" H 2350 4150 50  0000 C CNN
-F 2 "" H 2350 4300 50  0000 C CNN
-F 3 "" H 2350 4300 50  0000 C CNN
-	1    2350 4300
+P 2000 4400
+F 0 "#PWR013" H 2000 4150 50  0001 C CNN
+F 1 "GND" H 2000 4250 50  0000 C CNN
+F 2 "" H 2000 4400 50  0000 C CNN
+F 3 "" H 2000 4400 50  0000 C CNN
+	1    2000 4400
 	1    0    0    -1
 $EndComp
@@
 Text Label 8200 1800 0    60   ~ 0
 XTAL2
-Text Label 1550 3850 2    60   ~ 0
+Text Label 1200 3950 2    60   ~ 0
 XTAL1
-Text Label 2500 3850 0    60   ~ 0
+Text Label 2150 3950 0    60   ~ 0
 XTAL2
 Text Label 8200 2700 0    60   ~ 0
@@
 Connection ~ 5150 3400
 Wire Wire Line
-	1700 4250 1700 4300
-Wire Wire Line
-	2350 4250 2350 4300
-Wire Wire Line
-	1550 3850 1900 3850
-Wire Wire Line
-	1700 3850 1700 3950
-Wire Wire Line
-	2200 3850 2500 3850
-Wire Wire Line
-	2350 3850 2350 3950
+	1350 4350 1350 4400
+Wire Wire Line
+	2000 4350 2000 4400
+Wire Wire Line
+	1200 3950 1550 3950
+Wire Wire Line
+	1350 3950 1350 4050
+Wire Wire Line
+	1850 3950 2150 3950
+Wire Wire Line
+	2000 3950 2000 4050
 Wire Wire Line
 	8200 1800 7950 1800
 Wire Wire Line
 	7950 1700 8200 1700
-Connection ~ 1700 3850
-Connection ~ 2350 3850
+Connection ~ 1350 3950
+Connection ~ 2000 3950
 Wire Wire Line
 	7950 2700 8200 2700
@@
 Wire Wire Line
 	3850 1700 3300 1700
+Text Notes 2600 3550 0    39   Italic 0
+Copyright Sven Gregori 2015.\n\nThis documentation describes Open Hardware and is licensed under the\nCERN OHL v. 1.2. You may redistribute and modify this documentation\nunder the terms of the CERN OHL v.1.2. (http://ohwr.org/cernohl).\n\nThis documentation is distributed WITHOUT ANY EXPRESS OR IMPLIED\nWARRANTY, INCLUDING OF MERCHANTABILITY, SATISFACTORY QUALITY AND\nFITNESS FOR A PARTICULAR PURPOSE. Please see the CERN OHL v.1.2\nfor applicable conditions
 $EndSCHEMATC

Commit message: issue-#12: Initial version for Revision B hardware
Changed crystal value from 16MHz to 12MHz to match speed spec for
ATmega running at 3.3V. Changed LCD from Olimex Nokia 3310 with hard
to find connector to Nokia 5110 breakout board style so it can be
clipped directly into the PCB. Added LED based back light as well.
Adjusted some pin assignments for ongoing PCB design

Added BOM along the way.
Parts:
- removed C16: 1u, Capacitors_Tantalum_SMD:TantalC_SizeA_EIA-3216_HandSoldering, symbol C
- removed P4: Nokia 3310 LCD, LCD_Connectors:FPA-WZA201-08-LF, symbol CONN_01X08
- removed P5: LCD Backlight, SMD_Packages:SMD-2512_Pol, symbol CONN_01X02
- removed W1, W2, W3, W4, W5: TP, SMD_Packages:1Pin, symbol TEST_1P
- removed W7: TP, Pin_Headers:Pin_Header_Straight_1x01, symbol TEST_1P
- added D1, D2, D3, D4: LED, LEDs:LED_0805, symbol LED
- added Q1: 2N2222, TO_SOT_Packages_SMD:SOT-23, symbol Q_NPN_EBC
- added R16: 1k, Resistors_SMD:R_0805_HandSoldering, symbol R
- added R20: 0R, Resistors_SMD:R_0805_HandSoldering, symbol R
- added U2: Nokia_5110_LCD, Nokia_5110-3310_LCD:Nokia_5110-3310_LCD, symbol Nokia_5110_LCD
- C1, C2: footprint Capacitors_Tantalum_SMD:TantalC_SizeA_EIA-3216_HandSoldering -> Capacitors_Tantalum_SMD:CP_Tantalum_Case-A_EIA-3216-18_Hand
- P2: footprint Pin_Headers:Pin_Header_Straight_2x05 -> Connect:IDC_Header_Straight_10pins
- P3: value CONN_01X04 -> UART; footprint Pin_Headers:Pin_Header_Straight_1x04 -> Pin_Headers:Pin_Header_Straight_1x04_Pitch2.54mm
- R12, R13, R14: value 33k -> 100
- R15: value 100R -> 100
- SW1: renamed from SW2; value SW_PUSH -> Menu Minus
- SW2: renamed from SW4; value SW_PUSH -> Menu Select
- SW3: renamed from SW6; value SW_PUSH -> Menu Plus
- SW4: renamed from SW1; value SW_PUSH -> Chord I
- SW5: renamed from SW3; value SW_PUSH -> Chord V
- SW6: renamed from SW5; value SW_PUSH -> Chord vi
- SW7: value SW_PUSH -> Chord IV
- W1: renamed from W6; footprint Pin_Headers:Pin_Header_Straight_1x01 -> Pin_Headers:Pin_Header_Straight_1x01_Pitch2.54mm
- X1: value 16MHz -> 12MHz; footprint Crystals:crystal_FA238-TSX3225 -> Crystals:Crystal_SMD_HC49-SD_HandSoldering
- renumbered R18 to R17, R16 to R18, R17 to R19
Connections:
- net labels added: LCD_BACKLIGHT_PWM
- wire segments 161 -> 162
- no-connect marks 6 -> 5
Other:
- note added: "Copyright Sven Gregori 2017.\n\nThis documentation describes Open Hardware and is licensed under the\nCERN OHL v. 1.2. You may redistribute and modify this documentation\nunder the terms of the CERN OHL v.1.2. (http://ohwr.org/cernohl).\n\nThis documentation is distributed WITHOUT ANY EXPRESS OR IMPLIED\nWARRANTY, INCLUDING OF MERCHANTABILITY, SATISFACTORY QUALITY AND\nFITNESS FOR A PARTICULAR PU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"
- note removed: "Copyright Sven Gregori 2015.\n\nThis documentation describes Open Hardware and is licensed under the\nCERN OHL v. 1.2. You may redistribute and modify this documentation\nunder the terms of the CERN OHL v.1.2. (http://ohwr.org/cernohl).\n\nThis documentation is distributed WITHOUT ANY EXPRESS OR IMPLIED\nWARRANTY, INCLUDING OF MERCHANTABILITY, SATISFACTORY QUALITY AND\nFITNESS FOR A PARTICULAR PU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"
- moved on the sheet: P3, R17

Commit message: issue-#12: Completing Revision B schematic
Further pin adjustments to get better PCB routing done. Changed
programmer header from 10pin to 6pin for same reason.
Parts:
- removed P2: Programmer, Connect:IDC_Header_Straight_10pins, symbol CONN_02X05
- added P2: Programmer, Connect:IDC_Header_Straight_6pins, symbol CONN_02X03
- X1: footprint Crystals:Crystal_SMD_HC49-SD_HandSoldering -> Crystals:Crystal_SMD_HC49-SD
Connections:
- net labels added: Programmer
- wire segments 162 -> 166
Other:
- moved on the sheet: P3, R20
